Commit message: Increase max torque

File: thymio_description/urdf/base.urdf.xacro (robot description, xacro)
@@ -9,5 +9,5 @@
   <xacro:property name="wheel_axis" value="0.0935"/>
   <xacro:property name="wheel_radius" value="0.022"/>
-  <xacro:property name="wheel_torque" value="0.1"/>
+  <xacro:property name="wheel_torque" value="10.0"/>
   <xacro:property name="body_mass" value="0.2"/>
   <xacro:property name="wheel_mass" value="0.024"/>

Commit message: Added namespace

File: thymio_description/urdf/base.urdf.xacro (robot description, xacro)
@@ -66,13 +66,13 @@
     <xacro:wheel tf_prefix="${tf_prefix}" name="left" position="${wheel_axis * 0.5}" radius="${wheel_radius}" mass="${wheel_mass}" mu="$(arg left_wheel_mu)"/>
     <xacro:wheel tf_prefix="${tf_prefix}" name="right" position="${-wheel_axis * 0.5}" radius="${wheel_radius}" mass="${wheel_mass}" mu="$(arg right_wheel_mu)"/>
-    <xacro:proximity_sensor tf_prefix="${tf_prefix}" group="proximity" range_max="$(arg proximity_max_range)" resolution="$(arg proximity_resolution)" fov="$(arg proximity_fov)" name="center" xyz="0.08 0 0.035" rpy="0 0 0"/>
-    <xacro:proximity_sensor tf_prefix="${tf_prefix}" group="proximity" range_max="$(arg proximity_max_range)" resolution="$(arg proximity_resolution)" fov="$(arg proximity_fov)" name="center_left" xyz="0.0756 0.0261 0.035" rpy="0 0 0.33161"/>
-    <xacro:proximity_sensor tf_prefix="${tf_prefix}" group="proximity" range_max="$(arg proximity_max_range)" resolution="$(arg proximity_resolution)" fov="$(arg proximity_fov)" name="center_right" xyz="0.0756 -0.0261 0.035" rpy="0 0 -0.33161"/>
-    <xacro:proximity_sensor tf_prefix="${tf_prefix}" group="proximity" range_max="$(arg proximity_max_range)" resolution="$(arg proximity_resolution)" fov="$(arg proximity_fov)" name="left" xyz="0.063 0.0493 0.035" rpy="0 0 0.66323"/>
-    <xacro:proximity_sensor tf_prefix="${tf_prefix}" group="proximity" range_max="$(arg proximity_max_range)" resolution="$(arg proximity_resolution)" fov="$(arg proximity_fov)" name="right" xyz="0.063 -0.0493 0.035" rpy="0 0 -0.66323"/>
-    <xacro:proximity_sensor tf_prefix="${tf_prefix}" group="proximity" range_max="$(arg proximity_max_range)" resolution="$(arg proximity_resolution)" fov="$(arg proximity_fov)" name="rear_left" xyz="-0.03 0.0305 0.035" rpy="0 0 3.14159"/>
-    <xacro:proximity_sensor tf_prefix="${tf_prefix}" group="proximity" range_max="$(arg proximity_max_range)" resolution="$(arg proximity_resolution)" fov="$(arg proximity_fov)" name="rear_right" xyz="-0.03 -0.0305 0.035" rpy="0 0 3.14159"/>
-    <xacro:proximity_sensor tf_prefix="${tf_prefix}" group="ground" range_max="0.03" name="left" xyz="0.07157 0.01155 0.009" rpy="0 1.5708 0.24311"/>
-    <xacro:proximity_sensor tf_prefix="${tf_prefix}" group="ground" range_max="0.03" name="right" xyz="0.07157 -0.01155 0.009" rpy="0 1.5708 -0.24311"/>
+    <xacro:proximity_sensor ns="${_name}" tf_prefix="${tf_prefix}" group="proximity" range_max="$(arg proximity_max_range)" resolution="$(arg proximity_resolution)" fov="$(arg proximity_fov)" name="center" xyz="0.08 0 0.035" rpy="0 0 0"/>
+    <xacro:proximity_sensor ns="${_name}" tf_prefix="${tf_prefix}" group="proximity" range_max="$(arg proximity_max_range)" resolution="$(arg proximity_resolution)" fov="$(arg proximity_fov)" name="center_left" xyz="0.0756 0.0261 0.035" rpy="0 0 0.33161"/>
+    <xacro:proximity_sensor ns="${_name}" tf_prefix="${tf_prefix}" group="proximity" range_max="$(arg proximity_max_range)" resolution="$(arg proximity_resolution)" fov="$(arg proximity_fov)" name="center_right" xyz="0.0756 -0.0261 0.035" rpy="0 0 -0.33161"/>
+    <xacro:proximity_sensor ns="${_name}" tf_prefix="${tf_prefix}" group="proximity" range_max="$(arg proximity_max_range)" resolution="$(arg proximity_resolution)" fov="$(arg proximity_fov)" name="left" xyz="0.063 0.0493 0.035" rpy="0 0 0.66323"/>
+    <xacro:proximity_sensor ns="${_name}" tf_prefix="${tf_prefix}" group="proximity" range_max="$(arg proximity_max_range)" resolution="$(arg proximity_resolution)" fov="$(arg proximity_fov)" name="right" xyz="0.063 -0.0493 0.035" rpy="0 0 -0.66323"/>
+    <xacro:proximity_sensor ns="${_name}" tf_prefix="${tf_prefix}" group="proximity" range_max="$(arg proximity_max_range)" resolution="$(arg proximity_resolution)" fov="$(arg proximity_fov)" name="rear_left" xyz="-0.03 0.0305 0.035" rpy="0 0 3.14159"/>
+    <xacro:proximity_sensor ns="${_name}" tf_prefix="${tf_prefix}" group="proximity" range_max="$(arg proximity_max_range)" resolution="$(arg proximity_resolution)" fov="$(arg proximity_fov)" name="rear_right" xyz="-0.03 -0.0305 0.035" rpy="0 0 3.14159"/>
+    <xacro:proximity_sensor ns="${_name}" tf_prefix="${tf_prefix}" group="ground" range_max="0.03" name="left" xyz="0.07157 0.01155 0.009" rpy="0 1.5708 0.24311"/>
+    <xacro:proximity_sensor ns="${_name}" tf_prefix="${tf_prefix}" group="ground" range_max="0.03" name="right" xyz="0.07157 -0.01155 0.009" rpy="0 1.5708 -0.24311"/>
     <link name="${tf_prefix}laser_link"/>
     <joint name="${tf_prefix}base_laser_joint" type="fixed">
@@ -100,4 +100,5 @@
         <publish_odom_tf>true</publish_odom_tf>
         <robot_base_frame>${tf_prefix}base_link</robot_base_frame>
+        <namespace>${_name}</namespace>
       </plugin>
       <plugin name="joint_states" filename="libgazebo_ros_joint_state_publisher.so">
@@ -105,4 +106,5 @@
         <joint_name>${tf_prefix}left_wheel_joint</joint_name>
         <update_rate>$(arg odom_rate)</update_rate>
+        <namespace>${_name}</namespace>
       </plugin>
     </gazebo>
@@ -116,5 +118,5 @@
             <!-- Add namespace and remap the default topic -->
             <!-- TODO namespace is ignored! -->
-            <!-- <namespace>/ground_truth/${tf_prefix}</namespace> -->
+            <namespace>${_name}</namespace>
             <argument>odom:=ground_truth/odom</argument>
           </ros>

File: thymio_description/urdf/proximity_sensor.urdf.xacro (robot description, xacro)
@@ -1,5 +1,5 @@
 <?xml version="1.0"?>
 <robot xmlns:xacro="http://playerstage.sourceforge.net/gazebo/xmlschema/#xacro">
-  <xacro:macro name="proximity_sensor" params="group name xyz rpy tf_prefix='' update_rate:=10 range_min:=0.00 range_max:=0.12 resolution:=0.005 fov:=0.3">
+  <xacro:macro name="proximity_sensor" params="group name xyz rpy ns='' tf_prefix='' update_rate:=10 range_min:=0.00 range_max:=0.12 resolution:=0.005 fov:=0.3">
     <link name="${tf_prefix}${group}_${name}_link"/>
     <joint name="${tf_prefix}${group}_${name}_joint" type="fixed">
@@ -44,5 +44,5 @@
           <radiation_type>infrared</radiation_type>
           <ros>
-            <namespace>${tf_prefix}</namespace>
+            <namespace>${ns}</namespace>
             <argument>~/out:=${group}/${name}</argument>
           </ros>
