Commit message: Backported to ROS1 noetic

File: thymio_description/urdf/base.urdf.xacro (robot description, xacro)
@@ -1,22 +1,26 @@
 <?xml version="1.0"?>
 <robot xmlns:xacro="http://playerstage.sourceforge.net/gazebo/xmlschema/#xacro" name="thymio">
-  <xacro:include filename="wheel.urdf.xacro"/>
-  <xacro:include filename="proximity_sensor.urdf.xacro"/>
-  <xacro:include filename="imu.urdf.xacro"/>
-  <xacro:arg name="name" default=""/>
-  <xacro:arg name="left_wheel_mu" default="100.0"/>
-  <xacro:arg name="right_wheel_mu" default="100.0"/>
+  <xacro:include filename="$(find thymio_description)/urdf/wheel.urdf.xacro"/>
+  <xacro:include filename="$(find thymio_description)/urdf/proximity_sensor.urdf.xacro"/>
+  <xacro:include filename="$(find thymio_description)/urdf/imu.urdf.xacro"/>
+  <xacro:arg name="left_wheel_mu" default="1.0"/>
+  <xacro:arg name="right_wheel_mu" default="1.0"/>
   <xacro:property name="wheel_axis" value="0.0935"/>
+  <xacro:arg name="wheel_width" default="0.00015"/>
+  <xacro:property name="r_wheel_width" value="$(arg wheel_width)"/>
   <xacro:property name="wheel_radius" value="0.022"/>
-  <xacro:property name="wheel_torque" value="10.0"/>
+  <xacro:property name="wheel_torque" value="0.1"/>
+  <xacro:arg name="wheel_kp" default="100000"/>
   <xacro:property name="body_mass" value="0.2"/>
+  <xacro:arg name="body_kp" default="175000"/>
   <xacro:property name="wheel_mass" value="0.024"/>
   <xacro:arg name="proximity_max_range" default="0.12"/>
   <xacro:arg name="proximity_resolution" default="0.005"/>
   <xacro:arg name="proximity_fov" default="0.3"/>
+  <xacro:arg name="name" default=""/>
   <xacro:arg name="publish_ground_truth" default="false"/>
   <xacro:arg name="ground_truth_frame_id" default="/world"/>
   <xacro:arg name="ground_truth_update_rate" default="10.0"/>
-  <xacro:arg name="odom_rate" default="20.0"/>
+  <xacro:arg name="odom_max_rate" default="20.0"/>
   <xacro:property name="_name" value="$(arg name)"/>
   <xacro:if value="${_name != ''}">
@@ -27,5 +31,10 @@
   </xacro:if>
   <xacro:macro name="thymio">
-    <link name="${tf_prefix}base_link">
+    <link name="${tf_prefix}body_link">
+      <inertial>
+        <origin xyz="0.0243 0 0.0205"/>
+        <mass value="${body_mass}"/>
+        <inertia ixx="${0.002199 * body_mass}" ixy="0" ixz="${-0.000760 * body_mass}" iyy="${0.002639 * body_mass}" iyz="0" izz="${0.002526 * body_mass}"/>
+      </inertial>
       <collision>
         <origin xyz="0 0 0" rpy="0 0 0"/>
@@ -47,10 +56,5 @@
       </visual>
     </link>
-    <link name="${tf_prefix}body_link">
-      <inertial>
-        <origin xyz="0.0243 0 0.0315"/>
-        <mass value="${body_mass}"/>
-        <inertia ixx="${0.002199 * body_mass}" ixy="0" ixz="${-0.000760 * body_mass}" iyy="${0.002639 * body_mass}" iyz="0" izz="${0.002526 * body_mass}"/>
-      </inertial>
+    <link name="${tf_prefix}base_link">
     </link>
     <joint name="${tf_prefix}body_joint" type="fixed">
@@ -63,16 +67,18 @@
       <mu1>0.1</mu1>
       <mu2>0.1</mu2>
+      <kp>$(arg body_kp)</kp>
+      <kd>1</kd>
     </gazebo>
-    <xacro:wheel tf_prefix="${tf_prefix}" name="left" position="${wheel_axis * 0.5}" radius="${wheel_radius}" mass="${wheel_mass}" mu="$(arg left_wheel_mu)"/>
-    <xacro:wheel tf_prefix="${tf_prefix}" name="right" position="${-wheel_axis * 0.5}" radius="${wheel_radius}" mass="${wheel_mass}" mu="$(arg right_wheel_mu)"/>
-    <xacro:proximity_sensor ns="${_name}" tf_prefix="${tf_prefix}" group="proximity" range_max="$(arg proximity_max_range)" resolution="$(arg proximity_resolution)" fov="$(arg proximity_fov)" name="center" xyz="0.08 0 0.035" rpy="0 0 0"/>
-    <xacro:proximity_sensor ns="${_name}" tf_prefix="${tf_prefix}" group="proximity" range_max="$(arg proximity_max_range)" resolution="$(arg proximity_resolution)" fov="$(arg proximity_fov)" name="center_left" xyz="0.0756 0.0261 0.035" rpy="0 0 0.33161"/>
-    <xacro:proximity_sensor ns="${_name}" tf_prefix="${tf_prefix}" group="proximity" range_max="$(arg proximity_max_range)" resolution="$(arg proximity_resolution)" fov="$(arg proximity_fov)" name="center_right" xyz="0.0756 -0.0261 0.035" rpy="0 0 -0.33161"/>
-    <xacro:proximity_sensor ns="${_name}" tf_prefix="${tf_prefix}" group="proximity" range_max="$(arg proximity_max_range)" resolution="$(arg proximity_resolution)" fov="$(arg proximity_fov)" name="left" xyz="0.063 0.0493 0.035" rpy="0 0 0.66323"/>
-    <xacro:proximity_sensor ns="${_name}" tf_prefix="${tf_prefix}" group="proximity" range_max="$(arg proximity_max_range)" resolution="$(arg proximity_resolution)" fov="$(arg proximity_fov)" name="right" xyz="0.063 -0.0493 0.035" rpy="0 0 -0.66323"/>
-    <xacro:proximity_sensor ns="${_name}" tf_prefix="${tf_prefix}" group="proximity" range_max="$(arg proximity_max_range)" resolution="$(arg proximity_resolution)" fov="$(arg proximity_fov)" name="rear_left" xyz="-0.03 0.0305 0.035" rpy="0 0 3.14159"/>
-    <xacro:proximity_sensor ns="${_name}" tf_prefix="${tf_prefix}" group="proximity" range_max="$(arg proximity_max_range)" resolution="$(arg proximity_resolution)" fov="$(arg proximity_fov)" name="rear_right" xyz="-0.03 -0.0305 0.035" rpy="0 0 3.14159"/>
-    <xacro:proximity_sensor ns="${_name}" tf_prefix="${tf_prefix}" group="ground" range_max="0.03" name="left" xyz="0.07157 0.01155 0.009" rpy="0 1.5708 0.24311"/>
-    <xacro:proximity_sensor ns="${_name}" tf_prefix="${tf_prefix}" group="ground" range_max="0.03" name="right" xyz="0.07157 -0.01155 0.009" rpy="0 1.5708 -0.24311"/>
+    <xacro:wheel tf_prefix="${tf_prefix}" name="left" position="${wheel_axis * 0.5}" radius="${wheel_radius}" mass="${wheel_mass}" mu="$(arg left_wheel_mu)" kp="$(arg wheel_kp)" width="$(arg wheel_width)"/>
+    <xacro:wheel tf_prefix="${tf_prefix}" name="right" position="${-wheel_axis * 0.5}" radius="${wheel_radius}" mass="${wheel_mass}" mu="$(arg right_wheel_mu)" kp="$(arg wheel_kp)" width="$(arg wheel_width)"/>
+    <xacro:proximity_sensor tf_prefix="${tf_prefix}" group="proximity" range_max="$(arg proximity_max_range)" resolution="$(arg proximity_resolution)" fov="$(arg proximity_fov)" name="center" xyz="0.08 0 0.035" rpy="0 0 0"/>
+    <xacro:proximity_sensor tf_prefix="${tf_prefix}" group="proximity" range_max="$(arg proximity_max_range)" resolution="$(arg proximity_resolution)" fov="$(arg proximity_fov)" name="center_left" xyz="0.0756 0.0261 0.035" rpy="0 0 0.33161"/>
+    <xacro:proximity_sensor tf_prefix="${tf_prefix}" group="proximity" range_max="$(arg proximity_max_range)" resolution="$(arg proximity_resolution)" fov="$(arg proximity_fov)" name="center_right" xyz="0.0756 -0.0261 0.035" rpy="0 0 -0.33161"/>
+    <xacro:proximity_sensor tf_prefix="${tf_prefix}" group="proximity" range_max="$(arg proximity_max_range)" resolution="$(arg proximity_resolution)" fov="$(arg proximity_fov)" name="left" xyz="0.063 0.0493 0.035" rpy="0 0 0.66323"/>
+    <xacro:proximity_sensor tf_prefix="${tf_prefix}" group="proximity" range_max="$(arg proximity_max_range)" resolution="$(arg proximity_resolution)" fov="$(arg proximity_fov)" name="right" xyz="0.063 -0.0493 0.035" rpy="0 0 -0.66323"/>
+    <xacro:proximity_sensor tf_prefix="${tf_prefix}" group="proximity" range_max="$(arg proximity_max_range)" resolution="$(arg proximity_resolution)" fov="$(arg proximity_fov)" name="rear_left" xyz="-0.03 0.0305 0.035" rpy="0 0 3.14159"/>
+    <xacro:proximity_sensor tf_prefix="${tf_prefix}" group="proximity" range_max="$(arg proximity_max_range)" resolution="$(arg proximity_resolution)" fov="$(arg proximity_fov)" name="rear_right" xyz="-0.03 -0.0305 0.035" rpy="0 0 3.14159"/>
+    <xacro:proximity_sensor tf_prefix="${tf_prefix}" group="ground" range_max="0.03" name="left" xyz="0.07157 0.01155 0.0009" rpy="0 1.5708 0.24311"/>
+    <xacro:proximity_sensor tf_prefix="${tf_prefix}" group="ground" range_max="0.03" name="right" xyz="0.07157 -0.01155 0.0009" rpy="0 1.5708 -0.24311"/>
     <link name="${tf_prefix}laser_link"/>
     <joint name="${tf_prefix}base_laser_joint" type="fixed">
@@ -81,30 +87,27 @@
       <origin xyz="0 0 0.035"/>
     </joint>
-    <!-- We have a problem with xacro -->
-    <!-- <xacro:imu ns="$(arg name)"/> -->
+    <xacro:imu tf_prefix="${tf_prefix}"/>
     <!-- see https://github.com/ros-simulation/gazebo_ros_pkgs/blob/kinetic-devel/gazebo_plugins/src/gazebo_ros_diff_drive.cpp -->
     <gazebo>
       <plugin name="differential_drive_controller" filename="libgazebo_ros_diff_drive.so">
-        <odometry_source>0</odometry_source>
-        <always_on>true</always_on>
-        <update_rate>$(arg odom_rate)</update_rate>
-        <left_joint>${tf_prefix}left_wheel_joint</left_joint>
-        <right_joint>${tf_prefix}right_wheel_joint</right_joint>
-        <wheel_separation>${wheel_axis}</wheel_separation>
-        <wheel_diameter>${2 * wheel_radius}</wheel_diameter>
-        <max_wheel_torque>${wheel_torque}</max_wheel_torque>
-        <max_wheel_acceleration>0</max_wheel_acceleration>
-        <publish_odom>true</publish_odom>
-        <odometry_frame>${tf_prefix}odom</odometry_frame>
-        <publish_wheel_tf>true</publish_wheel_tf>
-        <publish_odom_tf>true</publish_odom_tf>
-        <robot_base_frame>${tf_prefix}base_link</robot_base_frame>
-        <namespace>${_name}</namespace>
-      </plugin>
-      <plugin name="joint_states" filename="libgazebo_ros_joint_state_publisher.so">
-        <joint_name>${tf_prefix}right_wheel_joint</joint_name>
-        <joint_name>${tf_prefix}left_wheel_joint</joint_name>
-        <update_rate>$(arg odom_rate)</update_rate>
-        <namespace>${_name}</namespace>
+        <legacyMode>false</legacyMode>
+        <rosDebugLevel>Info</rosDebugLevel>
+        <odometrySource>encoder</odometrySource>
+        <alwaysOn>true</alwaysOn>
+        <publishOdomTF>true</publishOdomTF>
+        <updateRate>$(arg odom_max_rate)</updateRate>
+        <leftJoint>${tf_prefix}left_wheel_joint</leftJoint>
+        <rightJoint>${tf_prefix}right_wheel_joint</rightJoint>
+        <wheelSeparation>${wheel_axis + 0 * r_wheel_width}</wheelSeparation>
+        <wheelDiameter>${2 * wheel_radius}</wheelDiameter>
+        <wheelTorque>${wheel_torque}</wheelTorque>
+        <wheelAcceleration>0</wheelAcceleration>
+        <commandTopic>cmd_vel</commandTopic>
+        <odometryTopic>odom</odometryTopic>
+        <odometryFrame>${tf_prefix}odom</odometryFrame>
+        <publishWheelJointState>true</publishWheelJointState>
+        <publishWheelTF>false</publishWheelTF>
+        <publishTf>true</publishTf>
+        <robotBaseFrame>${tf_prefix}base_link</robotBaseFrame>
       </plugin>
     </gazebo>
@@ -115,13 +118,8 @@
       <gazebo>
         <plugin name="ground_truth" filename="libgazebo_ros_p3d.so">
-          <ros>
-            <!-- Add namespace and remap the default topic -->
-            <!-- TODO namespace is ignored! -->
-            <namespace>${_name}</namespace>
-            <argument>odom:=ground_truth/odom</argument>
-          </ros>
-          <frame_name>$(arg ground_truth_frame_id)</frame_name>
-          <body_name>${tf_prefix}base_link</body_name>
-          <update_rate>$(arg ground_truth_update_rate)</update_rate>
+          <frameName>$(arg ground_truth_frame_id)</frameName>
+          <bodyName>${tf_prefix}base_link</bodyName>
+          <topicName>ground_truth/odom</topicName>
+          <updateRate>$(arg ground_truth_update_rate)</updateRate>
         </plugin>
       </gazebo>

File: thymio_description/urdf/imu.urdf.xacro (robot description, xacro)
@@ -1,45 +1,22 @@
 <?xml version="1.0"?>
 <robot xmlns:xacro="http://playerstage.sourceforge.net/gazebo/xmlschema/#xacro">
-  <xacro:macro name="imu" params="ns:='' tf_prefix:=''">
+  <xacro:macro name="imu" params="tf_prefix:=''">
     <gazebo reference="${tf_prefix}base_link">
+      <gravity>true</gravity>
       <sensor name="imu_sensor" type="imu">
         <always_on>true</always_on>
         <update_rate>16</update_rate>
         <visualize>true</visualize>
+        <topic>__default_topic__</topic>
+        <plugin filename="libgazebo_ros_imu_sensor.so" name="imu_plugin">
+          <topicName>imu</topicName>
+          <bodyName>${tf_prefix}base_link</bodyName>
+          <updateRateHZ>16</updateRateHZ>
+          <gaussianNoise>0.2646</gaussianNoise>
+          <xyzOffset>0 0 0</xyzOffset>
+          <rpyOffset>0 0 0</rpyOffset>
+          <frameName>${tf_prefix}base_link</frameName>
+        </plugin>
         <pose>0 0 0 0 0 0</pose>
-        <!-- There is a bug somewhere that make it ignore the next block, altough it passes formatting test
-          `gz sdf -v 1.5 -k ...`   -->
-          <!-- [ERROR] [launch]: Caught exception in launch (see debug for traceback): Unused block "linear_acceleration" -->
-        <imu>
-          <linear_acceleration>
-            <x>
-              <noise type="gaussian">
-                <mean>0.0</mean>
-                <stddev>0.2646</stddev>
-              </noise>
-            </x>
-            <y>
-              <noise type="gaussian">
-                <mean>0.0</mean>
-                <stddev>0.2646</stddev>
-              </noise>
-            </y>
-            <z>
-              <noise>
-                <type>gaussian</type>
-                <mean>0.0</mean>
-                <stddev>0.2646</stddev>
-              </noise>
-            </z>
-          </linear_acceleration>
-        </imu>
-        <plugin filename="libgazebo_ros_imu_sensor.so" name="imu_plugin">
-          <topic_name>${tf_prefix}imu</topic_name>
-          <body_name>${tf_prefix}base_link</body_name>
-          <frame_name>${tf_prefix}base_link</frame_name>
-          <ros>
-            <argument>~/out:=${tf_prefix}imu</argument>
-          </ros>
-        </plugin>
       </sensor>
     </gazebo>

File: thymio_description/urdf/proximity_sensor.urdf.xacro (robot description, xacro)
@@ -1,5 +1,5 @@
 <?xml version="1.0"?>
 <robot xmlns:xacro="http://playerstage.sourceforge.net/gazebo/xmlschema/#xacro">
-  <xacro:macro name="proximity_sensor" params="group name xyz rpy ns='' tf_prefix='' update_rate:=10 range_min:=0.00 range_max:=0.12 resolution:=0.005 fov:=0.3">
+  <xacro:macro name="proximity_sensor" params="group name xyz rpy tf_prefix:='' update_rate:=10 range_min:=0.01 range_max:=0.12 resolution:=0.005 fov:=0.3">
     <link name="${tf_prefix}${group}_${name}_link"/>
     <joint name="${tf_prefix}${group}_${name}_joint" type="fixed">
@@ -10,23 +10,8 @@
     <gazebo reference="${tf_prefix}${group}_${name}_link">
       <sensor name="${group}_${name}_sensor" type="ray">
-        <frame name="${tf_prefix}${group}_${name}_link"/>
         <visualize>true</visualize>
         <update_rate>${update_rate}</update_rate>
         <always_on>true</always_on>
         <ray>
-          <scan>
-            <horizontal>
-              <samples>1</samples>
-              <resolution>1</resolution>
-              <min_angle>-${fov / 2}</min_angle>
-              <max_angle>-${fov / 2}</max_angle>
-            </horizontal>
-            <vertical>
-              <samples>1</samples>
-              <resolution>1</resolution>
-              <min_angle>-${fov / 2}</min_angle>
-              <max_angle>-${fov / 2}</max_angle>
-            </vertical>
-          </scan>
           <range>
             <min>${range_min}</min>
@@ -34,18 +19,13 @@
             <resolution>${resolution}</resolution>
           </range>
-          <noise>
-            <type>gaussian</type>
-            <mean>0.0</mean>
-            <stddev>${resolution / 2}</stddev>
-          </noise>
         </ray>
-        <plugin name="${group}_${name}_controller" filename="libgazebo_ros_ray_sensor.so">
-          <!-- TODO: check if field `radiation` is still valid-->
-          <radiation_type>infrared</radiation_type>
-          <ros>
-            <namespace>${ns}</namespace>
-            <argument>~/out:=${group}/${name}</argument>
-          </ros>
-          <output_type>sensor_msgs/Range</output_type>
+        <plugin name="${group}_${name}_controller" filename="libgazebo_ros_range.so">
+          <alwaysOn>true</alwaysOn>
+          <updateRate>0</updateRate>
+          <frameName>${tf_prefix}${group}_${name}_link</frameName>
+          <topicName>${group}/${name}</topicName>
+          <radiation>infrared</radiation>
+          <fov>${fov}</fov>
+          <gaussianNoise>${resolution / 2}</gaussianNoise>
         </plugin>
       </sensor>

File: thymio_description/urdf/thymio.urdf.xacro (robot description, xacro)
@@ -1,5 +1,5 @@
 <?xml version="1.0"?>
 <robot name="thymio" xmlns:xacro="http://playerstage.sourceforge.net/gazebo/xmlschema/#xacro">
-  <xacro:include filename="base.urdf.xacro"/>
+  <xacro:include filename="$(find thymio_description)/urdf/base.urdf.xacro"/>
   <xacro:thymio/>
 </robot>

File: thymio_description/urdf/wheel.urdf.xacro (robot description, xacro)
@@ -1,5 +1,5 @@
 <?xml version="1.0"?>
 <robot xmlns:xacro="http://playerstage.sourceforge.net/gazebo/xmlschema/#xacro">
-  <xacro:macro name="wheel" params="name position tf_prefix='' mass:=0.024 mu:=100 radius:=0.022 width=0.015 max_speed=7.757">
+  <xacro:macro name="wheel" params="name position tf_prefix:='' mass:=0.024 mu:=100 radius:=0.022 width=0.015 max_speed=7.757 kp=10000">
     <link name="${tf_prefix}${name}_wheel_link">
       <inertial>
@@ -26,10 +26,12 @@
       <axis xyz="0 1 0"/>
       <origin xyz="0 ${position} ${radius}"/>
-      <limit velocity="${max_speed}" effort="0"/>
-      <dynamics damping="0.1" friction="0.1"/>
+      <!-- <limit velocity="${max_speed}" effort="0"/> -->
+      <!-- <dynamics damping="0.1" friction="0.1"/> -->
     </joint>
     <gazebo reference="${tf_prefix}${name}_wheel_link">
       <mu1>${mu}</mu1>
       <mu2>${mu / 2.0}</mu2>
+      <kp>${kp}</kp>
+      <kd>1</kd>
     </gazebo>
   </xacro:macro>
